Commit message: missing integration of apriltag from the top camera, all can be added in a single executable

File: models/pin_to_top_camera.urdf (robot description, URDF)
Before this commit: robot reachstacker, 8 links, 7 joints
Links:
- removed link laser
Joints:
- removed joint lidar_joint
- joint camera_endeffector_joint: origin xyz=0 0.050 -0.015 rpy=1.57 0 0 -> xyz=0 0.050 -0.015 rpy=-1.57 0 0
