Commit message: working on elbaorating the pariltag detection array, modified the urdf, tested in the lab, still achse 6 does not seems right

File: models/pin_to_ee_model.urdf (robot description, URDF)
Before this commit: robot reachstacker, 7 links, 6 joints
Joints:
- joint Achse7: limit lower=-0.005 upper=0.005 effort=1000.0 velocity=1000.0 -> lower=-0.040 upper=0.040 effort=1000.0 velocity=1000.0

File: models/shoulder_model.urdf (robot description, URDF)
Before this commit: robot reachstacker, 6 links, 5 joints
Joints:
- joint Achse7: limit lower=-0.005 upper=0.005 effort=1000.0 velocity=1000.0 -> lower=-0.040 upper=0.040 effort=1000.0 velocity=1000.0
